File: t-dsp_tac5212_audio_shield_adaptor.kicad_sch (KiCad schematic)
At the start: 212 parts, among them IC1 Logic Level Shifter - 74HCT2G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, J1 jumper, J10 JST-XH Connector, J11 JST-XH Connector, J12 RGB LED HEADEER, J13 Conn_01x02, J14 Conn_01x03, J15 Conn_01x01, J16 Conn_01x02, J17 Conn_02x04_Odd_Even, J18 Conn_02x02_Odd_Even, J19 Conn_01x01, J2 GROUND HEADER, J20 Conn_01x01, J21 jumper, J22 35RAPC4BV4, J23 35RAPC4BV4, J24 Conn_01x04, J25 PRT-14417, J26 73725-0110BLF, J27 Conn_01x04, J3 jumper, J4 jumper, J5 jumper, J6 jumper, J7 jumper, J8 PJRAS2X1S01X, J9 PJRAS2X1S01X, Q1 DMG2307L-7, Q2 DMG2307L-7, SW1 SW_SPST, SW2 TL1105WF160Q - 3.15mm actuator, SW3 SW_SPST, SW4 SW_SPST, SW5 RotaryEncoder_Switch_MP, SW6 TL1105WF160Q - 3.15mm actuator, SW7 TL1105WF160Q - 3.15mm actuator, SW8 TL1105WF160Q - 3.15mm actuator, T108 Tab, T109 Tab, T110 Tab, T111 Tab, U1 Teensy 4.1 - DEVKIT, U10 TPD4E02B04DQA, U2 ESP32-DevKitC - DEVKIT, U3 Power Mux & Protect - TPS2116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, U4 Optoisolators - H11L1SM - 6-S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, U5 Dual Buffer - SN74LVC2G125DCTR, U6 Dual Buffer - SN74LVC2G125DCTR, U7 Dual Buffer - SN74LVC2G125DCTR, U8 Dual Buffer - SN74LVC2G125DCTR, U9 Dual Buffer - 74HCT2G17GW,125

Commit message: v0.1: Finish routing, update board outline and revision
- Complete PCB routing and zone fills
- Add board outline footprint variants (-0.66mm offset)
- Update USB-A footprint to KiCad 9.0 format
- Fix schematic connections and capacitor orientation
- Correct project filename metadata
- Update 3D model
- Set REVISION to v0.1
Parts:
- #ESP32_SPI1, BAT1, C12, C13, C14, C15, C16, C17, C18, C19, C2, C20, C21, C22, C23, C27, C28, C29, C3, C30, C31, C32, C34, C35, C36, C37, C38, C39, C4, C5, CC1, CC2, D2, D3, D4, D5, ESP_I1, ETHERNET1, ETHERNET_J1, GPI1, IC1, J10, J11, J12, J13, J15, J16, J19, J2, J20, J22, J23, J24, J25, J26, J27, PWR1, PWR2, PWR3, Q1, Q2, R1, R10, R15, R16, R17, R18, R19, R2, R20, R21, R22, R23, R24, R27, R28, R29, R30, R31, R32, R33, R34, R35, R36, R37, R38, R39, R4, R40, R41, R42, R43, R44, R45, R46, R47, R48, R49, R5, R50, R51, R52, R53, R54, R7, R8, RLED1, RLED2, RLED3, TDM1, TDM2, TR2, TT2, T_PROG1, U10, U2, U3, U4, U5, U6, U7, U8, U9, USBC1, USB_DEVICE_1, board_outline2: now left out of the parts list
- C10, C40, C7, C9, J21, USBA1: now fitted; now in the parts list
- USB_HOST_1: now fitted
- board_outline1: footprint project_fp:audio_module_board_outline_50x34.5_d1_ADAPTOR -> project_fp:audio_module_board_outline_final_minus-.66_mod_long; now fitted; now in the parts list
Connections:
- net at C6.2, C7.2, J1.2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: now also HPTRS1.2, J1.1, J5.2, J_PHONE1.RN
- net at C8.2, C9.2, J3.1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: now also HPTRS1.5, J3.2, J4.1, J_PHONE1.TN
- net at MIC2.4 (LRCLK-WS-FS): now also MIC1.4 (LRCLK-WS-FS)
- net at MIC1.4 (LRCLK-WS-FS): no longer MIC2.4 (LRCLK-WS-FS)

Commit message: update
Parts:
- added J28: 6364372-2, project_fp:TE_Connectivity_6364372-2, symbol TE_Connectivity_6364372-2:6364372-2
- J21, board_outline1: now left out of the parts list
Connections:
- net at MIC2.4 (LRCLK-WS-FS): now also MIC1.4 (LRCLK-WS-FS)
- net at MIC1.4 (LRCLK-WS-FS): no longer MIC2.4 (LRCLK-WS-FS)
Changed lines of the file:
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@@
 		(exclude_from_sim no)
 		(in_bom no)
-		(on_board no)
+		(on_board yes)
 		(dnp yes)
 		(fields_autoplaced yes)
@@
 		(unit 1)
 		(exclude_from_sim no)
-		(in_bom yes)
+		(in_bom no)
 		(on_board yes)
 		(dnp no)
@@
 	)
 	(symbol
+		(lib_id "TE_Connectivity_6364372-2:6364372-2")
+		(at 883.92 529.59 0)
+		(unit 1)
+		(exclude_from_sim no)
+		(in_bom yes)
+		(on_board yes)
+		(dnp no)
+		(fields_autoplaced yes)
+		(property "Reference" "J28"
+			(at 897.89 532.1299 0)
+			(effects
+				(font
+					(size 1.524 1.524)
+				)
+				(justify left)
+			)
+		)
+		(property "Value" "6364372-2"
+			(at 897.89 534.6699 0)
+			(effects
+				(font
+					(size 1.524 1.524)
+				)
+				(justify left)
+			)
+		)
+		(property "Footprint" "project_fp:TE_Connectivity_6364372-2"
+			(at 883.92 529.59 0)
+			(effects
+				(font
+					(size 1.27 1.27)
+					(italic yes)
+				)
+				(hide yes)
+			)
+		)
+		(property "Datasheet" "6364372-2"
+			(at 883.92 529.59 0)
+			(effects
+				(font
+					(size 1.27 1.27)
+					(italic yes)
+				)
+				(hide yes)
+			)
+		)
+		(property "Description" ""
+			(at 883.92 529.59 0)
+			(effects
+				(font
+					(size 1.27 1.27)
+				)
+				(hide yes)
+			)
+		)
+		(pin "3"
+		)
+		(pin "1"
+		)
+		(pin "2"
+		)
+		(pin "4"
+		)
+		(instances
+			(project ""
+				(path "/6a0ff39d-771d-410f-9e7c-006586d81d16"
+					(reference "J28")
+					(unit 1)
+				)
+			)
+		)
+	)
+	(symbol
 		(lib_id "Device:LED")
 		(at 1123.95 501.65 180)
@@
 		(unit 1)
 		(exclude_from_sim no)
-		(in_bom yes)
+		(in_bom no)
 		(on_board yes)
 		(dnp no)
